Commit message: working finaly!!!

File: urdf/robot2_no_transmissions.urdf.xacro (robot description, xacro)
@@ -92,11 +92,10 @@
     <ros2_control name="testControl" type="system">
           <hardware>
-            <plugin>hardware_interface_wrappers/TransmissionWrapper</plugin>
-            <param name="wrapped_interface">fake_components/GenericSystem</param>
+            <plugin>test_hardware_interface_wrappers/TestableJointSystem</plugin>
           </hardware>
          <joint name="joint1">
                 <command_interface name="position"/>
-                <state_interface name="position">
-                </state_interface>
+                <command_interface name="velocity"/>
+                <state_interface name="position"/>
                 <state_interface name="velocity"/>
                 <state_interface name="effort"/>
@@ -104,6 +103,6 @@
             <joint name="joint2">
                 <command_interface name="position"/>
-                <state_interface name="position">
-                </state_interface>
+                <command_interface name="velocity"/>
+                <state_interface name="position"/>
                 <state_interface name="velocity"/>
                 <state_interface name="effort"/>
@@ -111,31 +110,9 @@
           <joint name="joint3">
                 <command_interface name="position"/>
-                <state_interface name="position">
-                </state_interface>
+                <command_interface name="velocity"/>
+                <state_interface name="position"/>
                 <state_interface name="velocity"/>
                 <state_interface name="effort"/>
             </joint>
-            <transmission name="transmission_scara">
-                  <plugin>transmission_interface/ScaraTransmission</plugin>
-                  <actuator name="actuator2" role="actuator2">
-                  </actuator>
-                  <actuator name="actuator3" role="actuator3">
-                  </actuator>
-                  <joint name="joint2" role="joint2">
-                    <offset>0.01236057350368102</offset>
-                    <mechanical_reduction>251.3274122872</mechanical_reduction>
-                  </joint>
-                  <joint name="joint3" role="joint3">
-                    <offset>0</offset>
-                    <mechanical_reduction>1.0</mechanical_reduction>
-                  </joint>
-                </transmission>
-                 <transmission name="transmission_joint1">
-                  <plugin>transmission_interface/BasicTransmission</plugin>
-                  <joint name="joint1" role="joint1">
-                    <mechanical_reduction>1.0</mechanical_reduction>
-                    <offset>0</offset>
-                  </joint>
-                </transmission>
         </ros2_control>
 </robot>
